File: batt.kicad_pcb (KiCad board)
At the start: 2 copper layers, 25 x 18 mm, 20 parts, among them J1 L+, J2 B+, J3 BATT, J4 B-, J5 V+, J6 L-, J7 USB_B_Micro, J8 V-, U1 FS312F-G, U2 FS8205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

Commit message: Various tweaks to schematic
Connections:
- net Net-(C1-Pad2) renamed /B-
