File: batt.sch (KiCad schematic (older format))
At the start: 20 parts, among them J1 L+, J2 B+, J3 BATT, J4 B-, J5 V+, J6 L-, J7 USB_B_Micro, J8 V-, U1 FS312F-G, U2 FS8205, U3 TP4056

Commit message: Various tweaks to schematic
Parts:
- J3: symbol Connector_Generic:Conn_01x02 -> Device:Battery_Cell
Connections:
- net B-: now reaches C1.2, J3.2 (-), J4.1 (Pin_1), U1.6 (GND), U2.1 (S1)
Other:
- note added: "Battery Charging"
- note added: "Battery Protection"
- moved on the sheet: C1, C2, C3, D1, J1, J2, J4, J5, J6, J7, J8, R1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
