File: led-addon/led-addon.sch (KiCad schematic (older format))
At the start: 19 parts, among them J1 VCC, J2 LED+, J3 LED-, J4 PWM, J5 STRT1, J6 GND, J8 STRT2, U1 PAM2804

Commit message: WIP
Parts:
- removed J4: PWM, Connector_PinHeader_2.54mm:PinHeader_1x02_P2.54mm_Vertical, symbol Connector_Generic:Conn_01x02
- added C3, C4: 100n, Capacitor_SMD:C_0603_1608Metric, symbol Device:C_Small
- added D2, D3: (no value), Diode_SMD:D_SOD-523, symbol Device:D_Small
- added R5: 100k, Resistor_SMD:R_0603_1608Metric, symbol Device:R_Small
- added RV1: 10k, Connector_PinHeader_2.54mm:PinHeader_1x03_P2.54mm_Vertical, symbol Device:R_POT_Small
- added SW1: PWR, Connector_PinHeader_2.54mm:PinHeader_1x03_P2.54mm_Vertical, symbol Switch:SW_SPDT
- added U2: MIC1557, Package_TO_SOT_SMD:SOT-23-5, symbol batt:MIC1557
Connections:
- net GND: now also C3.2, C4.2, U2.2 (GND)
- net VCC: now also C3.1, R5.1, SW1.2 (B), U2.4 (VS); no longer J1.1 (Pin_1)
- net at R4.2, U1.1 (EN): now also D2.1 (K), D3.2 (A), U2.5 (OUT)
- new net: J1.1 (Pin_1), SW1.1 (A)
- new net: C4.1, RV1.2, U2.1 (T/T)
- new net: R5.2, U2.3 (CS)
- new net: D3.1 (K), RV1.1
- new net: D2.2 (A), RV1.3
- no-connect marks 2 -> 3
Other:
- moved on the sheet: C1, C2, D1, J1, J2, J3, JP1, JP2, JP3, L1, R1, R2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
